File: smd/multi-avr/multi-avr.sch (KiCad schematic (older format))
At the start: 38 parts, among them J1 USB_B_Mini, SW1 SW_SPST, U1 ATmega32U4-AU, U2 ZIF, Y1 16MHz, Y2 16MHz

Commit message: Reworked schematic for the USB6 and correct caps
Parts:
- removed J1: USB_B_Mini, Connector_PinHeader_2.54mm:PinHeader_1x06_P2.54mm_Vertical, symbol Connector:USB_B_Mini
- removed R3: 10K, Resistor_SMD:R_0603_1608Metric, symbol Device:R_Small
- added C8: 4.7uF, Capacitor_SMD:C_0805_2012Metric, symbol Device:C_Small
- added R10, R9: 5.1K, Resistor_SMD:R_0805_2012Metric, symbol Device:R_Small
- added USB1: CLEAN-TYPE-C-31-M-12, Type-C:HRO-TYPE-C-31-M-12-HandSoldering, symbol Type-C:CLEAN-TYPE-C-31-M-12
- C1, C10, C2, C5: footprint Capacitor_SMD:C_0603_1608Metric -> Capacitor_SMD:C_0805_2012Metric; JLC C14663 -> C49678
- C11: footprint Capacitor_SMD:C_0603_1608Metric -> Capacitor_SMD:C_0805_2012Metric; JLC C19702 -> C15850
- C12: symbol Device:C_Small -> Device:CP1_Small
- C13: symbol Device:C_Small -> Device:CP1
- C14, C15, C6, C7: footprint Capacitor_SMD:C_0603_1608Metric -> Capacitor_SMD:C_0805_2012Metric; JLC C1653 -> C1804
- C3: JLC C14663 -> C49678
- C4: footprint Capacitor_SMD:C_0603_1608Metric -> Capacitor_SMD:C_0805_2012Metric; JLC (none) -> C1779
- C9: footprint Capacitor_SMD:C_0603_1608Metric -> Capacitor_SMD:C_0805_2012Metric; JLC C14663 -> C28323
- F1: JLC C163133 -> C163133
- R1, R2: footprint Resistor_SMD:R_0603_1608Metric -> Resistor_SMD:R_0805_2012Metric; JLC C23345 -> C17561
- R4: footprint Resistor_SMD:R_0603_1608Metric -> Resistor_SMD:R_0805_2012Metric; JLC C25804 -> C17414
- R5, R6, R7, R8: footprint Resistor_SMD:R_0603_1608Metric -> Resistor_SMD:R_0805_2012Metric; JLC C21190 -> C17513
- SW1: value SW_SPST -> PRG
Connections:
- net +5V: now also C12.1, C13.1; no longer C12.2, C13.2, C4.2, U1.42 (AREF)
- net GND: now also C12.2, C13.2, R4.2, C8.1, R10.2, R9.2, USB1.1 (GND), USB1.12 (GND), USB1.13 (SHIELD); no longer C12.1, C13.1, R4.1, SW1.1 (A)
- net ~S_RESET: now also SW1.1 (A)
- net at U1.33 (~HWB~/PE2): now also R4.1; no longer R4.2
- net USB_+5: now reaches D5.2 (A)
- net USB_+5: now also USB1.11 (VBUS), USB1.2 (VBUS)
- net X-: now reaches C7.1, U1.16 (XTAL2), Y1.3
- net X+: now reaches C6.1, U1.17 (XTAL1), Y1.1
- net D+: no longer names the net of R1.2
- net D+: now also C8.2, USB1.6 (DP1), USB1.8 (DP2)
- net D-: no longer names the net of R2.2
- net D-: now also C4.2, USB1.5 (DN2), USB1.7 (DN1)
- new net: R9.1, USB1.10 (CC2)
- new net: R10.1, USB1.4 (CC1)
- no-connect marks 31 -> 32
Other:
- note removed: "42"
- moved on the sheet: C3, C5, D3, D5, F1, R1, R2
